File: HARDWARE/Kicad Arena Luciano.kicad_pcb (KiCad board)
At the start: 2 copper layers, 46 parts, among them IC1 MC7805CD2TG, J1 BORNERA, J2 BORNERA, J4 BORNERA, J5 BORNERA, K3 SANYOU_SRD_Form_C, K6 SANYOU_SRD_Form_C, K7 SANYOU_SRD_Form_C, K8 SANYOU_SRD_Form_C, Q1 BC547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

Commit message: comi2
Parts:
- added J6: Conn_01x04_Pin, Connector_PinHeader_2.54mm:PinHeader_1x04_P2.54mm_Vertical, F.Cu at (59.4, 48.5)
- moved BORNERA1 33.7 mm to (50.8, 109.7), turned to -90 degrees
- moved R13 22.3 mm to (100.8, 109.8), turned to 0 degrees
- moved D9 21.3 mm to (101.0, 105.9), turned to 0 degrees
- moved C1 20.8 mm to (66.3, 112.4), turned to 180 degrees
- moved D7 19.0 mm to (100.8, 87.4), turned to 0 degrees
- moved R10 18.8 mm to (100.7, 91.4), turned to 0 degrees
- moved SW1 17.7 mm to (76.1, 114.9), turned to 180 degrees
- moved R15 17.2 mm to (95.1, 105.1), turned to 0 degrees
- moved R2 16.8 mm to (100.7, 73.8), turned to 0 degrees
- moved D1 16.3 mm to (100.8, 69.8), turned to 0 degrees
- moved R3 16.2 mm to (101.1, 55.8), turned to 0 degrees
- moved D3 16.0 mm to (101.2, 51.5), turned to 0 degrees
- moved IC1 16.0 mm to (64.7, 97.9), turned to 180 degrees
- moved K8 15.6 mm to (109.3, 107.8)
- moved J5 15.1 mm to (133.4, 102.8)
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Connections:
- D1 pad 2: ESP32 IO22 -> VCC
- D3 pad 2: ESP32 IO23 -> VCC
- D7 pad 2:  ESP32 IO21 -> VCC
- D9 pad 2: ESP32 IO19 -> VCC
- R10 pad 2: GND -> Net-(D8-A)
- R11 pad 1:  ESP32 IO21 ->  ESP32 IO17
- R13 pad 2: GND -> Net-(D10-A)
- R14 pad 1: ESP32 IO19 -> ESP32 IO16
- R2 pad 2: GND -> Net-(D4-A)
- R3 pad 2: GND -> Net-(D2-A)
- U7 pad 14: unconnected-(U7-GND1-Pad14) -> GND
- U7 pad 27: unconnected-(U7-IO16-Pad27) -> ESP32 IO16
- U7 pad 28: unconnected-(U7-IO17-Pad28) -> ESP32 IO17
- U7 pad 3: unconnected-(U7-SENSOR_VP-Pad3) -> Net-(J6-Pin_1)
- U7 pad 31: ESP32 IO19 -> unconnected-(U7-IO19-Pad31)
- U7 pad 32: unconnected-(U7-GND2-Pad32) -> GND
- U7 pad 33:  ESP32 IO21 -> unconnected-(U7-IO21-Pad33)
- U7 pad 4: unconnected-(U7-SENSOR_VN-Pad4) -> Net-(J6-Pin_2)
- U7 pad 5: unconnected-(U7-IO34-Pad5) -> Net-(J6-Pin_3)
- U7 pad 6: unconnected-(U7-IO35-Pad6) -> Net-(J6-Pin_4)
Routing:
- net VCC: track 494.4 -> 405.0 mm
- net ESP32 IO19: track 52.7 -> 0.00 mm
- net  ESP32 IO21: track 33.4 -> 0.00 mm
- net ESP32 IO16: track 0.00 -> 31.4 mm
- net Net-(J6-Pin_4): track 0.00 -> 30.5 mm
- net Net-(J6-Pin_3): track 0.00 -> 27.0 mm
- net Net-(J6-Pin_2): track 0.00 -> 23.4 mm
- net Net-(J6-Pin_1): track 0.00 -> 19.8 mm
- net  ESP32 IO17: track 0.00 -> 15.5 mm
- net Net-(BORNERA1-Pin_2): track 10.4 -> 25.3 mm
- net GND: track 13.4 -> 0.00 mm
- net Net-(D10-A): track 13.8 -> 23.5 mm
- net Net-(D8-A): track 12.7 -> 22.1 mm
- net ESP32 IO23: track 22.0 -> 13.8 mm
- net Net-(D4-A): track 15.5 -> 23.0 mm
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
Commit message: commit3
Parts:
- removed Q1, Q2, Q4, Q5: BC547, bc547:SOT95P230X110-3N
- added Q3: MMBT2222A, Package_TO_SOT_SMD:SOT-23, B.Cu at (95.5, 51.9)
- added Q6: MMBT2222A, Package_TO_SOT_SMD:SOT-23, B.Cu at (95.6, 69.8)
- added Q7: MMBT2222A, Package_TO_SOT_SMD:SOT-23, B.Cu at (95.5, 87.6)
- added Q8: MMBT2222A, Package_TO_SOT_SMD:SOT-23, B.Cu at (95.5, 105.7)
- moved R12 6.68 mm to (94.5, 93.3), turned to 90 degrees
- moved R6 6.56 mm to (94.5, 75.2), turned to 90 degrees
- moved R15 6.37 mm to (94.5, 111.4), turned to 90 degrees
- moved R4 5.72 mm to (94.5, 57.2), turned to 90 degrees
Routing:
- net Net-(U4-ET): track 8.95 -> 3.36 mm
- net Net-(U1-ET): track 8.77 -> 3.23 mm
- net Net-(U5-ET): track 8.26 -> 3.29 mm
- net Net-(U2-ET): track 8.01 -> 3.50 mm
- net Net-(D4-A): track 23.0 -> 24.5 mm
- net Net-(D8-A): track 22.1 -> 23.4 mm
- net Net-(Q6-E): track 4.56 -> 3.56 mm
- net Net-(D2-A): track 22.7 -> 23.7 mm
- net Net-(Q8-E): track 4.56 -> 3.92 mm
- net VCC: track 405.0 -> 404.4 mm
- net Net-(Q7-E): track 4.42 -> 3.89 mm

Commit message: commit4
Parts:
- U7: footprint ESP32:MODULE_ESP32-DEVKITC -> EESTN5:ESP32S
- moved Q8 0.57 mm to (95.4, 106.2), turned to 0 degrees
- moved Q6 0.14 mm to (95.4, 69.8), turned to 0 degrees
- turned Q3 to 0 degrees
- turned Q7 to 0 degrees
- turned U7 to -90 degrees
Connections:
- Q3 pad 1: Net-(D2-A) -> Net-(Q3-B)
- Q3 pad 2: Net-(Q3-E) -> GND
- Q3 pad 3: GND -> Net-(D2-A)
- Q6 pad 1: Net-(D4-A) -> Net-(Q6-B)
- Q6 pad 2: Net-(Q6-E) -> GND
- Q6 pad 3: GND -> Net-(D4-A)
- Q7 pad 1: Net-(D8-A) -> Net-(Q7-B)
- Q7 pad 2: Net-(Q7-E) -> GND
- Q7 pad 3: GND -> Net-(D8-A)
- Q8 pad 1: Net-(D10-A) -> Net-(Q8-B)
- Q8 pad 2: Net-(Q8-E) -> GND
- Q8 pad 3: GND -> Net-(D10-A)
- R12 pad 2: Net-(Q7-E) -> Net-(Q7-B)
- R15 pad 2: Net-(Q8-E) -> Net-(Q8-B)
- R4 pad 2: Net-(Q3-E) -> Net-(Q3-B)
- R6 pad 2: Net-(Q6-E) -> Net-(Q6-B)
Routing:
- net Net-(J6-Pin_4): track 30.5 -> 36.3 mm
- net Net-(J6-Pin_3): track 27.0 -> 31.1 mm
- net Net-(Q8-E): track 3.92 -> 0.00 mm
- net Net-(Q7-E): track 3.89 -> 0.00 mm
- net Net-(Q7-B): track 0.00 -> 3.86 mm
- net Net-(Q6-E): track 3.56 -> 0.00 mm
- net Net-(Q6-B): track 0.00 -> 3.54 mm
- net Net-(Q3-E): track 3.48 -> 0.00 mm
- net Net-(Q3-B): track 0.00 -> 3.47 mm
- net Net-(Q8-B): track 0.00 -> 3.34 mm
- net Net-(J6-Pin_2): track 23.4 -> 25.7 mm
- net Net-(D2-A): track 23.7 -> 25.6 mm
- net Net-(D8-A): track 23.4 -> 24.8 mm
- net Net-(D4-A): track 24.5 -> 25.8 mm
- net  ESP32 IO17: track 15.2 -> 16.5 mm
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