File: HARDWARE/Kicad Arena Luciano.kicad_sch (KiCad schematic)
At the start: 46 parts, among them IC1 MC7805CD2TG, J1 BORNERA, J2 BORNERA, J4 BORNERA, J5 BORNERA, K3 SANYOU_SRD_Form_C, K6 SANYOU_SRD_Form_C, K7 SANYOU_SRD_Form_C, K8 SANYOU_SRD_Form_C, Q1 BC547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

Commit message: comi2
Parts:
- added J6: Conn_01x04_Pin, Connector_PinHeader_2.54mm:PinHeader_1x04_P2.54mm_Vertical, symbol Connector:Conn_01x04_Pin
Connections:
- net ESP32 IO22: no longer D1.2 (A)
- net ESP32 IO23: no longer D3.2 (A)
- net GND: now also U7.14 (GND1), U7.32 (GND2); no longer R10.2, R13.2, R2.2, R3.2
- net VCC: now also D1.2 (A), D3.2 (A), D7.2 (A), D9.2 (A)
- net at D10.2 (A), K8.2, Q5.1 (C): now also R13.2
- net at D8.2 (A), K7.2, Q4.1 (C): now also R10.2
- net at D2.2 (A), K3.2, Q2.1 (C): now also R3.2
- net at D4.2 (A), K6.2, Q1.1 (C): now also R2.2
- net ESP32 IO16: now reaches U7.27 (IO16)
- net ESP32 IO16: now also R14.1
- net ESP32 IO17: now reaches U7.28 (IO17)
- net at U7.3 (SENSOR_VP): now also J6.1 (Pin_1)
- net at U7.4 (SENSOR_VN): now also J6.2 (Pin_2)
- net at U7.5 (IO34): now also J6.3 (Pin_3)
- net at U7.6 (IO35): now also J6.4 (Pin_4)
- net  ESP32 IO21 renamed  ESP32 IO17
- net  ESP32 IO17: no longer D7.2 (A)
- removed net ESP32 IO19: D9.2 (A), R14.1, U7.31 (IO19)
- net ESP32 IO21: no longer names the net of U7.33 (IO21)
- no-connect marks 6 -> 20
Other:
- moved on the sheet: D10, D2, D4, D8, R10, R13, R2, R3, U7

Commit message: commit3
Parts:
- removed Q1, Q2, Q4, Q5: BC547, bc547:SOT95P230X110-3N, symbol Transistor_BJT:BC547
- added Q3, Q6, Q7, Q8: MMBT2222A, Package_TO_SOT_SMD:SOT-23, symbol Transistor_BJT:MMBT2222A
Connections:
- net GND: now also Q3.3 (C), Q6.3 (C), Q7.3 (C), Q8.3 (C)
- net at D10.2 (A), K8.2, R13.2: now also Q8.1 (B)
- net at D8.2 (A), K7.2, R10.2: now also Q7.1 (B)
- net at R15.2: now also Q8.2 (E)
- net at D2.2 (A), K3.2, R3.2: now also Q3.1 (B)
- net at R4.2: now also Q3.2 (E)
- net at R6.2: now also Q6.2 (E)
- net at R12.2: now also Q7.2 (E)
- net at D4.2 (A), K6.2, R2.2: now also Q6.1 (B)

Commit message: commit4
Parts:
- U7: footprint ESP32:MODULE_ESP32-DEVKITC -> EESTN5:ESP32S
Connections:
- net GND: now also Q3.2 (E), Q6.2 (E), Q7.2 (E), Q8.2 (E); no longer Q3.3 (C), Q6.3 (C), Q7.3 (C), Q8.3 (C)
- net at D10.2 (A), K8.2, R13.2: now also Q8.3 (C); no longer Q8.1 (B)
- net at D8.2 (A), K7.2, R10.2: now also Q7.3 (C); no longer Q7.1 (B)
- net at R15.2: now also Q8.1 (B); no longer Q8.2 (E)
- net at D2.2 (A), K3.2, R3.2: now also Q3.3 (C); no longer Q3.1 (B)
- net at R4.2: now also Q3.1 (B); no longer Q3.2 (E)
- net at R12.2: now also Q7.1 (B); no longer Q7.2 (E)
- net at R6.2: now also Q6.1 (B); no longer Q6.2 (E)
- net at D4.2 (A), K6.2, R2.2: now also Q6.3 (C); no longer Q6.1 (B)
Other:
- moved on the sheet: Q3, Q6, Q7, Q8
Changed lines of the file:
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@@
 	)
 	(junction
+		(at 154.94 35.56)
+		(diameter 0)
+		(color 0 0 0 0)
+	)
+	(junction
 		(at 161.29 72.39)
 		(diameter 0)
@@
 	)
 	(junction
-		(at 154.94 35.56)
-		(diameter 0)
-		(color 0 0 0 0)
-	)
-	(junction
 		(at 147.32 20.32)
 		(diameter 0)
@@
 	)
 	(junction
-		(at 74.93 35.56)
+		(at 228.6 82.55)
 		(diameter 0)
 		(color 0 0 0 0)
 	)
 	(junction
-		(at 228.6 82.55)
+		(at 236.22 82.55)
 		(diameter 0)
 		(color 0 0 0 0)
 	)
 	(junction
-		(at 236.22 82.55)
+		(at 227.33 20.32)
 		(diameter 0)
 		(color 0 0 0 0)
 	)
 	(junction
-		(at 227.33 20.32)
+		(at 74.93 35.56)
 		(diameter 0)
 		(color 0 0 0 0)
@@
 	(wire
 		(pts
+			(xy 154.94 35.56) (xy 154.94 38.1)
+		)
+		(stroke
+			(width 0)
+			(type default)
+		)
+	)
+	(wire
+		(pts
 			(xy 72.39 82.55) (xy 78.74 82.55)
 		)
@@
 	(wire
 		(pts
-			(xy 102.87 77.47) (xy 102.87 81.28)
+			(xy 74.93 38.1) (xy 74.93 35.56)
 		)
 		(stroke
@@
 	(wire
 		(pts
-			(xy 67.31 43.18) (xy 69.85 43.18)
+			(xy 102.87 77.47) (xy 102.87 81.28)
 		)
 		(stroke
@@
 	(wire
 		(pts
-			(xy 227.33 43.18) (xy 229.87 43.18)
-		)
-		(stroke
-			(width 0)
-			(type default)
-		)
-	)
-	(wire
-		(pts
 			(xy 140.97 88.9) (xy 140.97 87.63)
 		)
@@
 	(wire
 		(pts
-			(xy 147.32 43.18) (xy 149.86 43.18)
-		)
-		(stroke
-			(width 0)
-			(type default)
-		)
-	)
-	(wire
-		(pts
 			(xy 62.23 35.56) (xy 67.31 35.56)
 		)
@@
 	(wire
 		(pts
-			(xy 228.6 90.17) (xy 231.14 90.17)
-		)
-		(stroke
-			(width 0)
-			(type default)
-		)
-	)
-	(wire
-		(pts
 			(xy 27.94 113.03) (xy 31.75 113.03)
 		)
@@
 	(symbol
 		(lib_id "Transistor_BJT:MMBT2222A")
-		(at 74.93 40.64 270)
+		(at 72.39 43.18 0)
 		(unit 1)
 		(exclude_from_sim no)
@@
 		(on_board yes)
 		(dnp no)
-		(fields_autoplaced yes)
 		(property "Reference" "Q3"
-			(at 74.93 46.99 90)
+			(at 77.47 41.9099 0)
 			(effects
 				(font
 					(size 1.27 1.27)
 				)
+				(justify left)
 			)
 		)
 		(property "Value" "MMBT2222A"
-			(at 74.93 49.53 90)
+			(at 77.47 44.45 0)
 			(effects
 				(font
 					(size 1.27 1.27)
 				)
+				(justify left)
 			)
 		)
 		(property "Footprint" "Package_TO_SOT_SMD:SOT-23"
-			(at 73.025 45.72 0)
+			(at 77.47 45.085 0)
 			(effects
 				(font
@@
 		)
 		(property "Datasheet" "https://assets.nexperia.com/documents/data-sheet/MMBT2222A.pdf"
-			(at 74.93 40.64 0)
+			(at 72.39 43.18 0)
 			(effects
 				(font
@@
 		)
 		(property "Description" "600mA Ic, 40V Vce, NPN Transistor, SOT-23"
-			(at 74.93 40.64 0)
+			(at 72.39 43.18 0)
 			(effects
 				(font
@@
 	(symbol
 		(lib_id "Transistor_BJT:MMBT2222A")
-		(at 234.95 40.64 270)
+		(at 232.41 43.18 0)
 		(unit 1)
 		(exclude_from_sim no)
@@
 		(fields_autoplaced yes)
 		(property "Reference" "Q7"
-			(at 234.95 46.99 90)
+			(at 237.49 41.9099 0)
 			(effects
 				(font
 					(size 1.27 1.27)
 				)
+				(justify left)
 			)
 		)
 		(property "Value" "MMBT2222A"
-			(at 234.95 49.53 90)
+			(at 237.49 44.4499 0)
 			(effects
 				(font
 					(size 1.27 1.27)
 				)
+				(justify left)
 			)
 		)
 		(property "Footprint" "Package_TO_SOT_SMD:SOT-23"
-			(at 233.045 45.72 0)
+			(at 237.49 45.085 0)
 			(effects
 				(font
@@
 		)
 		(property "Datasheet" "https://assets.nexperia.com/documents/data-sheet/MMBT2222A.pdf"
-			(at 234.95 40.64 0)
+			(at 232.41 43.18 0)
 			(effects
 				(font
@@
 		)
 		(property "Description" "600mA Ic, 40V Vce, NPN Transistor, SOT-23"
-			(at 234.95 40.64 0)
+			(at 232.41 43.18 0)
 			(effects
 				(font
@@
 	(symbol
 		(lib_id "Transistor_BJT:MMBT2222A")
-		(at 236.22 87.63 270)
+		(at 233.68 90.17 0)
 		(unit 1)
 		(exclude_from_sim no)
@@
 		(fields_autoplaced yes)
 		(property "Reference" "Q8"
-			(at 236.22 93.98 90)
+			(at 238.76 88.8999 0)
 			(effects
 				(font
 					(size 1.27 1.27)
 				)
+				(justify left)
 			)
 		)
 		(property "Value" "MMBT2222A"
-			(at 236.22 96.52 90)
+			(at 238.76 91.4399 0)
 			(effects
 				(font
 					(size 1.27 1.27)
 				)
+				(justify left)
 			)
 		)
 		(property "Footprint" "Package_TO_SOT_SMD:SOT-23"
-			(at 234.315 92.71 0)
+			(at 238.76 92.075 0)
 			(effects
 				(font
@@
 		)
 		(property "Datasheet" "https://assets.nexperia.com/documents/data-sheet/MMBT2222A.pdf"
-			(at 236.22 87.63 0)
+			(at 233.68 90.17 0)
 			(effects
 				(font
@@
 		)
 		(property "Description" "600mA Ic, 40V Vce, NPN Transistor, SOT-23"
-			(at 236.22 87.63 0)
+			(at 233.68 90.17 0)
 			(effects
 				(font
@@
 	(symbol
 		(lib_id "power:GND")
-		(at 80.01 43.18 0)
+		(at 74.93 48.26 0)
 		(unit 1)
 		(exclude_from_sim no)
@@
 		(dnp no)
 		(property "Reference" "#PWR03"
-			(at 80.01 49.53 0)
+			(at 74.93 54.61 0)
 			(effects
 				(font
@@
 		)
 		(property "Value" "GND"
-			(at 80.01 46.99 0)
+			(at 74.93 52.07 0)
 			(effects
 				(font
@@
 		)
 		(property "Footprint" ""
-			(at 80.01 43.18 0)
+			(at 74.93 48.26 0)
 			(effects
 				(font
@@
 		)
 		(property "Datasheet" ""
-			(at 80.01 43.18 0)
+			(at 74.93 48.26 0)
 			(effects
 				(font
@@
 		)
 		(property "Description" "Power symbol creates a global label with name \"GND\" , ground"
-			(at 80.01 43.18 0)
+			(at 74.93 48.26 0)
 			(effects
 				(font
@@
 	(symbol
 		(lib_id "power:GND")
-		(at 160.02 43.18 0)
+		(at 154.94 48.26 0)
 		(unit 1)
 		(exclude_from_sim no)
@@
 		(dnp no)
 		(property "Reference" "#PWR08"
-			(at 160.02 49.53 0)
+			(at 154.94 54.61 0)
 			(effects
 				(font
@@
 		)
 		(property "Value" "GND"
-			(at 160.02 46.99 0)
+			(at 154.94 52.07 0)
 			(effects
 				(font
@@
 		)
 		(property "Footprint" ""
-			(at 160.02 43.18 0)
+			(at 154.94 48.26 0)
 			(effects
 				(font
@@
 		)
 		(property "Datasheet" ""
-			(at 160.02 43.18 0)
+			(at 154.94 48.26 0)
 			(effects
 				(font
@@
 		)
 		(property "Description" "Power symbol creates a global label with name \"GND\" , ground"
-			(at 160.02 43.18 0)
+			(at 154.94 48.26 0)
 			(effects
 				(font
@@
 	(symbol
 		(lib_id "power:GND")
-		(at 241.3 90.17 0)
+		(at 236.22 95.25 0)
 		(unit 1)
 		(exclude_from_sim no)
@@
 		(dnp no)
 		(property "Reference" "#PWR020"
-			(at 241.3 96.52 0)
+			(at 236.22 101.6 0)
 			(effects
 				(font
@@
 		)
 		(property "Value" "GND"
-			(at 241.3 93.98 0)
+			(at 236.22 99.06 0)
 			(effects
 				(font
@@
 		)
 		(property "Footprint" ""
-			(at 241.3 90.17 0)
+			(at 236.22 95.25 0)
 			(effects
 				(font
@@
 		)
 		(property "Datasheet" ""
-			(at 241.3 90.17 0)
+			(at 236.22 95.25 0)
 			(effects
 				(font
@@
 		)
 		(property "Description" "Power symbol creates a global label with name \"GND\" , ground"
-			(at 241.3 90.17 0)
+			(at 236.22 95.25 0)
 			(effects
 				(font
@@
 	(symbol
 		(lib_id "power:GND")
-		(at 240.03 43.18 0)
+		(at 234.95 48.26 0)
 		(unit 1)
 		(exclude_from_sim no)
@@
 		(dnp no)
 		(property "Reference" "#PWR016"
-			(at 240.03 49.53 0)
+			(at 234.95 54.61 0)
 			(effects
 				(font
@@
 		)
 		(property "Value" "GND"
-			(at 240.03 46.99 0)
+			(at 234.95 52.07 0)
 			(effects
 				(font
@@
 		)
 		(property "Footprint" ""
-			(at 240.03 43.18 0)
+			(at 234.95 48.26 0)
 			(effects
 				(font
@@
 		)
 		(property "Datasheet" ""
-			(at 240.03 43.18 0)
+			(at 234.95 48.26 0)
 			(effects
 				(font
@@
 		)
 		(property "Description" "Power symbol creates a global label with name \"GND\" , ground"
-			(at 240.03 43.18 0)
+			(at 234.95 48.26 0)
 			(effects
 				(font
@@
 	(symbol
 		(lib_id "Transistor_BJT:MMBT2222A")
-		(at 154.94 40.64 270)
+		(at 152.4 43.18 0)
 		(unit 1)
 		(exclude_from_sim no)
@@
 		(dnp no)
 		(property "Reference" "Q6"
-			(at 154.94 46.99 90)
+			(at 158.75 43.18 90)
 			(effects
 				(font
@@
 		)
 		(property "Value" "MMBT2222A"
-			(at 154.94 50.8 90)
+			(at 162.56 43.18 90)
 			(effects
 				(font
@@
 		)
 		(property "Footprint" "Package_TO_SOT_SMD:SOT-23"
-			(at 153.035 45.72 0)
+			(at 157.48 45.085 0)
 			(effects
 				(font
@@
 		)
 		(property "Datasheet" "https://assets.nexperia.com/documents/data-sheet/MMBT2222A.pdf"
-			(at 154.94 40.64 0)
+			(at 152.4 43.18 0)
 			(effects
 				(font
@@
 		)
 		(property "Description" "600mA Ic, 40V Vce, NPN Transistor, SOT-23"
-			(at 154.94 40.64 0)
+			(at 152.4 43.18 0)
 			(effects
 				(font
@@
 			)
 		)
-		(property "Footprint" "ESP32:MODULE_ESP32-DEVKITC"
+		(property "Footprint" "EESTN5:ESP32S"
 			(at 52.07 90.17 0)
 			(effects
