File: Amplificador/AMPLI.kicad_sch (KiCad schematic)
At the start: 18 parts, among them J1 Conn_01x03_Pin, J2 Screw_Terminal_01x02, J3 Screw_Terminal_01x02, U1 TDA2050

Commit message: commit20
Parts:
- removed J1: Conn_01x03_Pin, symbol Connector:Conn_01x03_Pin
- added SW1: SW_DPST_x2, Connector_PinHeader_2.54mm:PinHeader_1x03_P2.54mm_Vertical, symbol Switch:SW_DPST_x2
- J2, J3: footprint TerminalBlock:TerminalBlock_Xinya_XY308-2.54-2P_1x02_P2.54mm_Horizontal -> EESTN5:BORNERA2_AZUL
Connections:
- net at RV1.1: now also SW1.2 (B)
- net at J3.2 (Pin_2): now also SW1.1 (A)
Other:
- moved on the sheet: J3
